File: plasma/plasma/plasma.kicad_pcb (KiCad board)
At the start: 2 copper layers, 215.8 x 70.2 mm, 24 parts, among them X6 14-Pin Cable

Commit message: Final commit before disassociating from combined repo
Parts:
- removed 12V DC-DC Power Buck: ~, Transistor_Power_Module:Weewooday Adjustable LM2596S DC-DC Buck Converter
- removed X6: 14-Pin Cable, Package_DIP:DIP-14_W10.16mm
- added 12V DC to 5V DC Power Buck: ~, Transistor_Power_Module:Weewooday Adjustable LM2596S DC-DC Buck Converter, F.Cu at (152.5, 116.2)
- added R10: 8 Ω, PLASMA_PARTS:R_Axial_DIN0411_L60.0mm_D10mm_P15.24mm_Horizontal 20Watt 8Ohm, F.Cu at (47.7, 155.7)
- added R11: 8 Ω, PLASMA_PARTS:R_Axial_DIN0411_L60.0mm_D10mm_P15.24mm_Horizontal 20Watt 8Ohm, F.Cu at (120.4, 155.8)
- added R12: 8 Ω, PLASMA_PARTS:R_Axial_DIN0411_L60.0mm_D10mm_P15.24mm_Horizontal 20Watt 8Ohm, F.Cu at (192.8, 155.9)
- added R13: 1 Ω, PLASMA_PARTS:R_Axial_DIN0411_L60.0mm_D10mm_P15.24mm_Horizontal 20Watt 8Ohm, F.Cu at (193.1, 127.9)
- added R14: 1 Ω, PLASMA_PARTS:R_Axial_DIN0411_L60.0mm_D10mm_P15.24mm_Horizontal 20Watt 8Ohm, F.Cu at (258.9, 122.8)
- added R15: 1 Ω, PLASMA_PARTS:R_Axial_DIN0411_L60.0mm_D10mm_P15.24mm_Horizontal 20Watt 8Ohm, F.Cu at (168.5, 107.8)
- added R16: 1 Ω, PLASMA_PARTS:R_Axial_DIN0411_L60.0mm_D10mm_P15.24mm_Horizontal 20Watt 8Ohm, F.Cu at (192.9, 136.6)
- added R5: 1 Ω, PLASMA_PARTS:R_Axial_DIN0411_L60.0mm_D10mm_P15.24mm_Horizontal 20Watt 8Ohm, F.Cu at (47.8, 127.8)
- added R6: 8 Ω, PLASMA_PARTS:R_Axial_DIN0411_L60.0mm_D10mm_P15.24mm_Horizontal 20Watt 8Ohm, F.Cu at (47.8, 119.0)
- added R7: 8 Ω, PLASMA_PARTS:R_Axial_DIN0411_L60.0mm_D10mm_P15.24mm_Horizontal 20Watt 8Ohm, F.Cu at (47.8, 145.9)
- added R8: 8 Ω, PLASMA_PARTS:R_Axial_DIN0411_L60.0mm_D10mm_P15.24mm_Horizontal 20Watt 8Ohm, F.Cu at (120.4, 146.0)
- added R9: 1 Ω, PLASMA_PARTS:R_Axial_DIN0411_L60.0mm_D10mm_P15.24mm_Horizontal 20Watt 8Ohm, F.Cu at (192.9, 146.1)
- added X1 - 14-Pin Cable: 14-Pin Cable, Package_DIP:DIP-14_W10.16mm, F.Cu at (249.2, 86.7)
- R1: value 17 Ω -> 1 Ω; footprint Resistor_THT:R_Axial_DIN0411_L9.9mm_D3.6mm_P15.24mm_Horizontal -> PLASMA_PARTS:R_Axial_DIN0411_L60.0mm_D10mm_P15.24mm_Horizontal 20Watt 8Ohm
- R2: value 1.5 Ω -> 1 Ω; footprint Resistor_THT:R_Axial_DIN0411_L9.9mm_D3.6mm_P15.24mm_Horizontal -> PLASMA_PARTS:R_Axial_DIN0411_L60.0mm_D10mm_P15.24mm_Horizontal 20Watt 8Ohm
- R3: value 22 Ω -> 8 Ω; footprint Resistor_THT:R_Axial_DIN0411_L9.9mm_D3.6mm_P15.24mm_Horizontal -> PLASMA_PARTS:R_Axial_DIN0411_L60.0mm_D10mm_P15.24mm_Horizontal 20Watt 8Ohm
- R4: value 3.3 Ω -> 1 Ω; footprint Resistor_THT:R_Axial_DIN0411_L9.9mm_D3.6mm_P15.24mm_Horizontal -> PLASMA_PARTS:R_Axial_DIN0411_L60.0mm_D10mm_P15.24mm_Horizontal 20Watt 8Ohm
- moved R4 139.9 mm to (47.8, 136.7)
- moved R2 90.4 mm to (120.4, 127.8)
- moved R1 90.2 mm to (120.4, 119.0)
- moved ? 86.8 mm to (267.0, 158.7)
- moved ? 85.4 mm to (266.5, 50.3)
- moved R3 72.6 mm to (120.3, 136.6)
- moved G*** 65.3 mm to (215.7, 59.8)
- moved G*** 41.0 mm to (214.7, 95.9)
- moved ? 31.8 mm to (155.3, 73.4)
- moved ? 30.3 mm to (32.1, 158.9)
- moved ? 28.7 mm to (33.7, 49.9)
- moved D2 26.3 mm to (178.4, 73.4)
- moved ? 24.9 mm to (155.4, 90.2)
- moved ? 24.9 mm to (50.0, 112.0)
- moved ? 24.9 mm to (147.4, 63.6)
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Connections:
- net /GND renamed Net-(D1-K)
- ? pad 1: Net-(P1-+12VDC) -> +5V
- ? pad 1: (no net) -> -12V
- ? pad 1: (no net) -> -5V
- ? pad 1: Net-(P1-+12VDC) -> +12V
- D1 pad 2: Net-(D1-A) -> -5V
- D2 pad 2: Net-(D2-A) -> +5V
- R1 pad 1: Net-(P1-+12VDC) -> +5V
- R1 pad 2: /+12VDC -> Net-(R1-Pad2)
- R2 pad 1: Net-(P1--12VDC) -> +5V
- R2 pad 2: /-12VDC -> Net-(R1-Pad2)
- R3 pad 1: Net-(D1-A) -> +5V
- R3 pad 2: /-5VDC -> Net-(R1-Pad2)
- R4 pad 1: Net-(D2-A) -> -5V
- R4 pad 2: /+5VDC -> Net-(R16-Pad1)
Routing:
- net -5V: track 0.00 -> 222.1 mm
- net Net-(P1-+12VDC): track 185.0 -> 0.00 mm
- net Net-(P1--12VDC): track 170.7 -> 0.00 mm
- net +5V: track 0.00 -> 146.9 mm
- net Net-(D1-A): track 133.1 -> 0.00 mm
- net +12V: track 0.00 -> 114.9 mm
- net /+5VDC: track 105.0 -> 0.00 mm
- net Net-(R16-Pad1): track 0.00 -> 102.7 mm
- net /-5VDC: track 97.0 -> 0.00 mm, vias 4 -> 0
- net -12V: track 0.00 -> 94.3 mm
- net Net-(R15-Pad2): track 0.00 -> 89.8 mm
- net Net-(R12-Pad2): track 0.00 -> 83.2 mm
- net /-12VDC: track 75.4 -> 0.00 mm, vias 5 -> 0
- net Net-(R16-Pad2): track 0.00 -> 61.0 mm, vias 0 -> 1
- net Net-(D2-A): track 55.4 -> 0.00 mm
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Other:
- board size 215.8 x 70.2 mm -> 242.9 x 117.4 mm
- board text added: "Note: This product has no affiliation with the original Sphere Corporation"
- board text added: "Parts List P1 12V DC-DC Power Buck D1/D2 IN4001 R1/R2/R4 R5/R9/R13 1Ω 20W rated R14/R15/R16 R3/R6/R7 R8/R10/R11 8Ω 20W rated R12 Sockets: 3.5mm 12DC centre -ve receptacle 14 pin connector Miscellaneous: 1 x 14 Pin ribbon cable 4 x M3 20+6mm standoffs 4 x M3 x 6mm screws"
- board text added: "SERIAL NUMBER : PLS/B/__________________________"
- board text removed: "Note: This product has no afiliation with the original Sphere Corporation"
- board text removed: "Parts List P1 12V DC=DC Power Buck D1/D2 IN4001 x 2 R1 17Ω R2 1.5Ω R3 22Ω R4 3.3Ω Sockets: 3.5mm 12DC centre -ve receptacle 14 pin connector"
- board text removed: "SERIAL NUMBER : PLS/A/__________________________"
