File: plasma/plasma/plasma.kicad_sch (KiCad schematic)
At the start: 8 parts, among them X1 14-Pin Cable

Commit message: Final commit before disassociating from combined repo
Parts:
- removed R3: 22 Ω, Resistor_THT:R_Axial_DIN0411_L9.9mm_D3.6mm_P15.24mm_Horizontal, symbol Device:R_Small
- added R10: 8 Ω, PLASMA_PARTS:R_Axial_DIN0411_L60.0mm_D10mm_P15.24mm_Horizontal 20Watt 8Ohm, symbol Device:R_Small
- added R11, R12, R6, R7, R8: 8 Ω, Resistor_THT:R_Axial_DIN0411_L9.9mm_D3.6mm_P15.24mm_Horizontal, symbol Device:R_Small
- added R13, R14, R15, R16, R4, R5, R9: 1 Ω, Resistor_THT:R_Axial_DIN0411_L9.9mm_D3.6mm_P15.24mm_Horizontal, symbol Device:R_Small
- 12V DC to 5V DC Power Buck: renamed from P1
- R1: value 17 Ω -> 1 Ω
- R2: value 1.5 Ω -> 1 Ω
- R3: renamed from R4; value 3.3 Ω -> 8 Ω
- X1 - 14-Pin Cable: renamed from X1
Connections:
- net +12VDC: now also R9.2; no longer R1.2
- net +5VDC: no longer R3.2, X1 - 14-Pin Cable.13, X1 - 14-Pin Cable.14, X1 - 14-Pin Cable.6, X1 - 14-Pin Cable.7
- net -12VDC: no longer R2.2, X1 - 14-Pin Cable.12, X1 - 14-Pin Cable.5
- net -5VDC: no longer X1 - 14-Pin Cable.11, X1 - 14-Pin Cable.4
- net GND: no longer D1.1 (K), D2.1 (K), X1 - 14-Pin Cable.1, X1 - 14-Pin Cable.2, X1 - 14-Pin Cable.8, X1 - 14-Pin Cable.9
- net at R1.1: now also 12V DC to 5V DC Power Buck.3 (+5VDC), D2.2 (A), R2.1, R3.1; no longer 12V DC to 5V DC Power Buck.1 (+12VDC)
- net at 12V DC to 5V DC Power Buck.4 (-5VDC), D1.2 (A): now also R4.1, R5.1, R6.1
- net -12V: now reaches 12V DC to 5V DC Power Buck.2 (-12VDC)
- net -12V: now also R10.1; no longer R2.1
- new net: R16.1, R4.2, R5.2, R6.2
- new net: R10.2, R11.1
- new net: R11.2, R12.1
- new net: R1.2, R13.1, R2.2, R3.2
- new net: D1.1 (K), D2.1 (K), X1 - 14-Pin Cable.1, X1 - 14-Pin Cable.2, X1 - 14-Pin Cable.8, X1 - 14-Pin Cable.9
- new net: R7.2, R8.1
- new net: R8.2, R9.1
- new net: R14.2, R15.1
- new net: R15.2, X1 - 14-Pin Cable.13, X1 - 14-Pin Cable.14, X1 - 14-Pin Cable.6, X1 - 14-Pin Cable.7
- new net: R12.2, X1 - 14-Pin Cable.12, X1 - 14-Pin Cable.5
- new net: R16.2, X1 - 14-Pin Cable.11, X1 - 14-Pin Cable.4
- new net: R13.2, R14.1
- new net +12V: 12V DC to 5V DC Power Buck.1 (+12VDC), R7.1
Other:
- note added: "0.2"
- note added: "11-MAR-2024"
- note added: "Updated with increased wattage resistors"
- moved on the sheet: D1, D2, R3
